File: Secondcansat.sch (KiCad schematic (older format))
At the start: 53 parts, among them IC1 XBP9B-XCWT-001, J1 OpenlogBreakout, J10 SDA, J11 5V, J12 Tx, J13 Rx, J14 Battery_Holder_keystone 1079, J15 USB_B_Mini, J16 coinBattery, J2 Camera, J3 Pressure_MS5607, J4 Debugger, J6 CAM-M8Q-GPS, J7 GND, J8 SCL, J9 3v, Q1 Q_PMOS_DMG2305UX-13DIDKR-ND, Q2 Q_NMOS_BSS138, Q3 Q_NMOS_BSS138, Q4 Q_NMOS_BSS138, U1 VR_TPS7A7001DDAR

Commit message: Wired up I2C sensors
Parts:
- added R? (x2): 10kohm, Resistor_SMD:R_0603_1608Metric_Pad1.05x0.95mm_HandSolder, symbol Device:R
Connections:
- wire segments 112 -> 124
Changed lines of the file:
@@
 F1 "IMU.sch" 50
 $EndSheet
-Text GLabel 3350 5300 2    50   Input ~ 0
+Text GLabel 3750 5300 2    50   Input ~ 0
 SCL
-Text GLabel 3350 5200 2    50   Input ~ 0
+Text GLabel 3750 5200 2    50   Input ~ 0
 SDA
 $Comp
@@
 	1    0    0    -1
 $EndComp
+$Comp
+L power:GND #PWR?
+U 1 1 5DCD0C96
+P 9700 4000
+F 0 "#PWR?" H 9700 3750 50  0001 C CNN
+F 1 "GND" H 9700 3850 50  0000 C CNN
+F 2 "" H 9700 4000 50  0001 C CNN
+F 3 "" H 9700 4000 50  0001 C CNN
+	1    9700 4000
+	0    1    1    0
+$EndComp
+Wire Wire Line
+	9850 4000 9750 4000
+Wire Wire Line
+	9850 3900 9750 3900
+Wire Wire Line
+	9750 3900 9750 4000
+Connection ~ 9750 4000
+Wire Wire Line
+	9750 4000 9700 4000
+$Comp
+L power:+5V #PWR?
+U 1 1 5DCDA59C
+P 9700 3600
+F 0 "#PWR?" H 9700 3450 50  0001 C CNN
+F 1 "+5V" H 9700 3740 50  0000 C CNN
+F 2 "" H 9700 3600 50  0001 C CNN
+F 3 "" H 9700 3600 50  0001 C CNN
+	1    9700 3600
+	0    -1   -1   0
+$EndComp
+Wire Wire Line
+	9700 3600 9850 3600
+$Comp
+L power:+3.3V #PWR?
+U 1 1 5DCDEF61
+P 3800 4900
+F 0 "#PWR?" H 3800 4750 50  0001 C CNN
+F 1 "+3.3V" H 3800 5040 50  0000 C CNN
+F 2 "" H 3800 4900 50  0001 C CNN
+F 3 "" H 3800 4900 50  0001 C CNN
+	1    3800 4900
+	0    1    1    0
+$EndComp
+Wire Wire Line
+	3750 5300 3650 5300
+Connection ~ 3450 5200
+Wire Wire Line
+	3450 5200 3750 5200
+Wire Wire Line
+	3350 5200 3450 5200
+$Comp
+L Device:R R?
+U 1 1 5DCE8943
+P 3450 5050
+F 0 "R?" H 3520 5096 50  0000 L CNN
+F 1 "10kohm" H 3520 5005 50  0000 L CNN
+F 2 "Resistor_SMD:R_0603_1608Metric_Pad1.05x0.95mm_HandSolder" V 3380 5050 50  0001 C CNN
+F 3 "~" H 3450 5050 50  0001 C CNN
+	1    3450 5050
+	1    0    0    -1
+$EndComp
+$Comp
+L Device:R R?
+U 1 1 5DCEE7A3
+P 3650 5150
+F 0 "R?" H 3720 5196 50  0000 L CNN
+F 1 "10kohm" H 3720 5105 50  0000 L CNN
+F 2 "Resistor_SMD:R_0603_1608Metric_Pad1.05x0.95mm_HandSolder" V 3580 5150 50  0001 C CNN
+F 3 "~" H 3650 5150 50  0001 C CNN
+	1    3650 5150
+	1    0    0    -1
+$EndComp
+Connection ~ 3650 5300
+Wire Wire Line
+	3650 5300 3350 5300
+Wire Wire Line
+	3450 4900 3650 4900
+Wire Wire Line
+	3650 5000 3650 4900
+Connection ~ 3650 4900
+Wire Wire Line
+	3650 4900 3800 4900
+Text GLabel 9850 3700 0    50   Input ~ 0
+SDA
+Text GLabel 9850 3800 0    50   Input ~ 0
+SCL
 $EndSCHEMATC

Commit message: pressure sensor footprint
Parts:
- removed C1, C5: 10uF, Capacitor_SMD:C_1206_3216Metric_Pad1.42x1.75mm_HandSolder, symbol Device:CP1
- removed C14, C3: 5uF, Capacitor_SMD:C_0603_1608Metric_Pad1.05x0.95mm_HandSolder, symbol Device:C
- removed C2, C4: 100nF, Capacitor_SMD:C_0603_1608Metric_Pad1.05x0.95mm_HandSolder, symbol Device:C
- removed C6: 10uF, Capacitor_SMD:C_0805_2012Metric_Pad1.15x1.40mm_HandSolder, symbol Device:C
- removed C7, C8: 1uF, Capacitor_SMD:C_0603_1608Metric_Pad1.05x0.95mm_HandSolder, symbol Device:C
- removed C9: 50uF, Capacitor_SMD:C_1206_3216Metric_Pad1.42x1.75mm_HandSolder, symbol Device:C
- removed IC1: XBP9B-XCWT-001, CanSAT2ndtry:XBP9BXCWT001_2, symbol Secondcansat-rescue:XBP9B-XCWT-001-Cansat-rescue
- removed IMU1: BN0055breakout, CanSAT2ndtry:BNO055breakout, symbol Secondcansat-rescue:IMUbreakout-Cansat-rescue
- removed J1: OpenlogBreakout, Connector_PinSocket_2.54mm:PinSocket_1x06_P2.54mm_Vertical, symbol Secondcansat-rescue:Conn_01x06-Connector_Generic
- removed J10: SDA, Connector_PinSocket_2.54mm:PinSocket_1x01_P2.54mm_Vertical, symbol Connector_Generic:Conn_01x01
- removed J11: 5V, Connector_PinSocket_2.54mm:PinSocket_1x01_P2.54mm_Vertical, symbol Connector_Generic:Conn_01x01
- removed J12: Tx, Connector_PinSocket_2.54mm:PinSocket_1x01_P2.54mm_Vertical, symbol Connector_Generic:Conn_01x01
- removed J13: Rx, Connector_PinSocket_2.54mm:PinSocket_1x01_P2.54mm_Vertical, symbol Connector_Generic:Conn_01x01
- removed J14: Battery_Holder_keystone 1079, CanSAT2ndtry:BatteryHolder, symbol Secondcansat-rescue:Battery_Holder-Cansat-rescue
- removed J15: USB_B_Mini, CanSAT2ndtry:USB-Mini, symbol Connector:USB_B_Mini
- removed J16: coinBattery, CanSAT2ndtry:coin_Battery_120591-1, symbol Secondcansat-rescue:coinBattery-Cansat-rescue
- removed J2: Camera, Connector_PinSocket_2.54mm:PinSocket_1x03_P2.54mm_Vertical, symbol Connector_Generic:Conn_01x03
- removed J3: Pressure_MS5607, CanSAT2ndtry:MS5607, symbol Secondcansat-rescue:Pressure_MS5607-Cansat-rescue
- removed J4: Debugger, Connector_PinSocket_1.27mm:PinSocket_2x03_P1.27mm_Vertical, symbol Connector_Generic:Conn_02x03_Odd_Even
- removed J6: CAM-M8Q-GPS, CanSAT2ndtry:CAM-M8Q, symbol Secondcansat-rescue:CAM-M8Q-GPS-Cansat-rescue
- removed J7: GND, Connector_PinSocket_2.54mm:PinSocket_1x01_P2.54mm_Vertical, symbol Connector_Generic:Conn_01x01
- removed J8: SCL, Connector_PinSocket_2.54mm:PinSocket_1x01_P2.54mm_Vertical, symbol Connector_Generic:Conn_01x01
- removed J9: 3v, Connector_PinSocket_2.54mm:PinSocket_1x01_P2.54mm_Vertical, symbol Connector_Generic:Conn_01x01
- removed L1, L2: 10uH, Inductor_SMD:L_0805_2012Metric_Pad1.15x1.40mm_HandSolder, symbol pspice:INDUCTOR
- removed MCU1: ATxmega128A4U-AU, CanSAT2ndtry:ATXMEGA128A4U-AU, symbol Secondcansat-rescue:ATxmega128A4U-AU-MCU_Microchip_ATmega
- removed Q1: Q_PMOS_DMG2305UX-13DIDKR-ND, Package_TO_SOT_SMD:SOT-23, symbol Device:Q_PMOS_DGS
- removed Q2, Q3, Q4: Q_NMOS_BSS138, Package_TO_SOT_SMD:SOT-23, symbol Device:Q_NMOS_DGS
- removed R1: 274kohm, Resistor_SMD:R_1206_3216Metric, symbol Device:R
- removed R10, R8: 2kohm, Capacitor_SMD:C_0805_2012Metric, symbol Device:R
- removed R11, R17, R20, R5, R6, R7, R? (x2): 10kohm, Resistor_SMD:R_0603_1608Metric_Pad1.05x0.95mm_HandSolder, symbol Device:R
- removed R18, R19: 220ohm, Resistor_SMD:R_0603_1608Metric_Pad1.05x0.95mm_HandSolder, symbol Device:R
- removed R2: 30Kohm, Resistor_SMD:R_0805_2012Metric_Pad1.15x1.40mm_HandSolder, symbol Device:R
- removed R9: 5kohm, Capacitor_SMD:C_0805_2012Metric, symbol Device:R
- removed Servo1: Servo_Adafruit_1142, Connector_PinSocket_2.54mm:PinSocket_1x03_P2.54mm_Vertical, symbol Connector_Generic:Conn_01x03
- removed TH1: Therm_NXRT15WB473FA3A016, Connector_PinSocket_2.54mm:PinSocket_2x01_P2.54mm_Vertical, symbol Device:Thermistor
- removed U1: VR_TPS7A7001DDAR, CanSAT2ndtry:VR_TPS7A7001DDAR, symbol Secondcansat-rescue:VR_TPS7A7001DDAR-Cansat-rescue
- removed U?: SPS30, symbol valkyrie_symbols:SPS30
- removed VR1: VR__TLV75533PDBVR, CanSAT2ndtry:VR_296-50411-1-ND, symbol Secondcansat-rescue:VR__TLV75533PDBVR-Cansat-rescue
- removed buzzer1: buzzer_MAS803Q, Connector_PinSocket_2.54mm:PinSocket_1x02_P2.54mm_Vertical, symbol Connector_Generic:Conn_02x01
Connections:
- net labels removed: +3.3V, +5V, +6V, ADC_A1, CSB, GND, INT, MCUAVCC, MCUVCC, MISO, MOSI, MoterRIN1, MoterRIN2, MotorFIN1, MotorFIN2, PDICLK, PDIDATA, PWM, RX_PD2, RX_PD6, SCL, SCLK, SDA, TC_PD0, TX_PD3, TX_PD7, Therm_ADCA0, USART_RX_PC2, USART_TX_PC3, cameraon
- wire segments 124 -> 0
- no-connect marks 7 -> 0

Commit message: footprints for pmos and 5VR
Parts:
- added C1, C5: 10uF, Capacitor_SMD:C_1206_3216Metric_Pad1.42x1.75mm_HandSolder, symbol Device:CP1
- added C14, C3: 5uF, Capacitor_SMD:C_0603_1608Metric_Pad1.05x0.95mm_HandSolder, symbol Device:C
- added C2, C4: 100nF, Capacitor_SMD:C_0603_1608Metric_Pad1.05x0.95mm_HandSolder, symbol Device:C
- added C6: 10uF, Capacitor_SMD:C_0805_2012Metric_Pad1.15x1.40mm_HandSolder, symbol Device:C
- added C7, C8: 1uF, Capacitor_SMD:C_0603_1608Metric_Pad1.05x0.95mm_HandSolder, symbol Device:C
- added C9: 50uF, Capacitor_SMD:C_1206_3216Metric_Pad1.42x1.75mm_HandSolder, symbol Device:C
- added IC1: XBP9B-XCWT-001, CanSAT2ndtry:XBP9BXCWT001_2, symbol Secondcansat-rescue:XBP9B-XCWT-001-Cansat-rescue
- added IMU1: BN0055breakout, CanSAT2ndtry:BNO055breakout, symbol Secondcansat-rescue:IMUbreakout-Cansat-rescue
- added J1: OpenlogBreakout, Connector_PinSocket_2.54mm:PinSocket_1x06_P2.54mm_Vertical, symbol Secondcansat-rescue:Conn_01x06-Connector_Generic
- added J10: SDA, Connector_PinSocket_2.54mm:PinSocket_1x01_P2.54mm_Vertical, symbol Connector_Generic:Conn_01x01
- added J11: 5V, Connector_PinSocket_2.54mm:PinSocket_1x01_P2.54mm_Vertical, symbol Connector_Generic:Conn_01x01
- added J12: Tx, Connector_PinSocket_2.54mm:PinSocket_1x01_P2.54mm_Vertical, symbol Connector_Generic:Conn_01x01
- added J13: Rx, Connector_PinSocket_2.54mm:PinSocket_1x01_P2.54mm_Vertical, symbol Connector_Generic:Conn_01x01
- added J14: Battery_Holder_keystone 1079, CanSAT2ndtry:BatteryHolder, symbol Secondcansat-rescue:Battery_Holder-Cansat-rescue
- added J15: USB_B_Mini, CanSAT2ndtry:USB-Mini, symbol Connector:USB_B_Mini
- added J16: coinBattery, CanSAT2ndtry:coin_Battery_120591-1, symbol Secondcansat-rescue:coinBattery-Cansat-rescue
- added J2: Camera, Connector_PinSocket_2.54mm:PinSocket_1x03_P2.54mm_Vertical, symbol Connector_Generic:Conn_01x03
- added J3: Pressure_MS5607, CanSAT2ndtry:MS5607, symbol Secondcansat-rescue:Pressure_MS5607-Cansat-rescue
- added J4: Debugger, Connector_PinSocket_1.27mm:PinSocket_2x03_P1.27mm_Vertical, symbol Connector_Generic:Conn_02x03_Odd_Even
- added J6: CAM-M8Q-GPS, CanSAT2ndtry:CAM-M8Q, symbol Secondcansat-rescue:CAM-M8Q-GPS-Cansat-rescue
- added J7: GND, Connector_PinSocket_2.54mm:PinSocket_1x01_P2.54mm_Vertical, symbol Connector_Generic:Conn_01x01
- added J8: SCL, Connector_PinSocket_2.54mm:PinSocket_1x01_P2.54mm_Vertical, symbol Connector_Generic:Conn_01x01
- added J9: 3v, Connector_PinSocket_2.54mm:PinSocket_1x01_P2.54mm_Vertical, symbol Connector_Generic:Conn_01x01
- added L1, L2: 10uH, Inductor_SMD:L_0805_2012Metric_Pad1.15x1.40mm_HandSolder, symbol pspice:INDUCTOR
- added MCU1: ATxmega128A4U-AU, CanSAT2ndtry:ATXMEGA128A4U-AU, symbol Secondcansat-rescue:ATxmega128A4U-AU-MCU_Microchip_ATmega
- added Q1: Q_PMOS_DMG2305UX-13DIDKR-ND, Package_TO_SOT_SMD:SOT-23, symbol Device:Q_PMOS_DGS
- added Q2, Q3, Q4: Q_NMOS_BSS138, Package_TO_SOT_SMD:SOT-23, symbol Device:Q_NMOS_DGS
- added R1: 274kohm, Resistor_SMD:R_1206_3216Metric, symbol Device:R
- added R10, R8: 2kohm, Capacitor_SMD:C_0805_2012Metric, symbol Device:R
- added R11, R17, R20, R5, R6, R7: 10kohm, Resistor_SMD:R_0603_1608Metric_Pad1.05x0.95mm_HandSolder, symbol Device:R
- added R18, R19: 220ohm, Resistor_SMD:R_0603_1608Metric_Pad1.05x0.95mm_HandSolder, symbol Device:R
- added R2: 30Kohm, Resistor_SMD:R_0805_2012Metric_Pad1.15x1.40mm_HandSolder, symbol Device:R
- added R9: 5kohm, Capacitor_SMD:C_0805_2012Metric, symbol Device:R
- added Servo1: Servo_Adafruit_1142, Connector_PinSocket_2.54mm:PinSocket_1x03_P2.54mm_Vertical, symbol Connector_Generic:Conn_01x03
- added TH1: Therm_NXRT15WB473FA3A016, Connector_PinSocket_2.54mm:PinSocket_2x01_P2.54mm_Vertical, symbol Device:Thermistor
- added U1: VR_TPS7A7001DDAR, CanSAT2ndtry:VR_TPS7A7001DDAR, symbol Secondcansat-rescue:VR_TPS7A7001DDAR-Cansat-rescue
- added U?: SPS30, symbol valkyrie_symbols:SPS30
- added VR1: VR__TLV75533PDBVR, CanSAT2ndtry:VR_296-50411-1-ND, symbol Secondcansat-rescue:VR__TLV75533PDBVR-Cansat-rescue
- added buzzer1: buzzer_MAS803Q, Connector_PinSocket_2.54mm:PinSocket_1x02_P2.54mm_Vertical, symbol Connector_Generic:Conn_02x01
Connections:
- net labels added: +3.3V, +5V, +6V, ADC_A1, CSB, GND, INT, MCUAVCC, MCUVCC, MISO, MOSI, MoterRIN1, MoterRIN2, MotorFIN1, MotorFIN2, PDICLK, PDIDATA, PWM, RX_PD2, RX_PD6, SCL, SCLK, SDA, TC_PD0, TX_PD3, TX_PD7, Therm_ADCA0, USART_RX_PC2, USART_TX_PC3, cameraon
- wire segments 0 -> 111
- no-connect marks 0 -> 7

Commit message: Differential pressure sensor
Parts:
- added C10: 100nF, Capacitor_SMD:C_0603_1608Metric_Pad1.05x0.95mm_HandSolder, symbol Device:C
- added U2: SAir_Speed_DP32-125PA-TR-250PCS, symbol valkyrie_symbols:SAir_Speed_DP32-125PA-TR-250PCS
- gave numbers to parts that had none: 1
Connections:
- wire segments 111 -> 132
- no-connect marks 7 -> 12
Changed lines of the file:
@@
 	8700 1600 8700 1650
 $Comp
-L power:GND #PWR?
+L power:GND #PWR0109
 U 1 1 5CA36EA2
 P 8700 1450
-F 0 "#PWR?" H 8700 1200 50  0001 C CNN
+F 0 "#PWR0109" H 8700 1200 50  0001 C CNN
 F 1 "GND" V 8705 1322 50  0000 R CNN
 F 2 "" H 8700 1450 50  0001 C CNN
@@
 $EndComp
 $Comp
-L valkyrie_symbols:SPS30 U?
+L valkyrie_symbols:SPS30 U3
 U 1 1 5DC9BC9E
 P 10100 3800
-F 0 "U?" H 10100 4100 50  0000 C CNN
+F 0 "U3" H 10100 4100 50  0000 C CNN
 F 1 "SPS30" H 10100 3500 50  0000 C CNN
 F 2 "" H 10200 3900 50  0001 C CNN
@@
 Wire Wire Line
 	1300 850  1300 1500
+$Comp
+L valkyrie_symbols:SAir_Speed_DP32-125PA-TR-250PCS U2
+U 1 1 5DE1D27B
+P 4950 1450
+F 0 "U2" H 5691 1646 50  0000 L CNN
+F 1 "SAir_Speed_DP32-125PA-TR-250PCS" H 4400 1000 50  0000 L CNN
+F 2 "" H 4900 1500 50  0001 C CNN
+F 3 "" H 4900 1500 50  0001 C CNN
+	1    4950 1450
+	1    0    0    -1
+$EndComp
+$Comp
+L power:GND #PWR0110
+U 1 1 5DE1D687
+P 4300 1650
+F 0 "#PWR0110" H 4300 1400 50  0001 C CNN
+F 1 "GND" H 4305 1477 50  0000 C CNN
+F 2 "" H 4300 1650 50  0001 C CNN
+F 3 "" H 4300 1650 50  0001 C CNN
+	1    4300 1650
+	1    0    0    -1
+$EndComp
+Wire Wire Line
+	4350 1100 4300 1100
+Wire Wire Line
+	4300 1100 4300 1350
+Wire Wire Line
+	4300 1550 4350 1550
+Connection ~ 4300 1550
+Wire Wire Line
+	4300 1550 4300 1650
+Wire Wire Line
+	4350 1350 4300 1350
+Connection ~ 4300 1350
+Wire Wire Line
+	4300 1350 4300 1550
+$Comp
+L power:GND #PWR0111
+U 1 1 5DE28572
+P 5700 1650
+F 0 "#PWR0111" H 5700 1400 50  0001 C CNN
+F 1 "GND" H 5705 1477 50  0000 C CNN
+F 2 "" H 5700 1650 50  0001 C CNN
+F 3 "" H 5700 1650 50  0001 C CNN
+	1    5700 1650
+	1    0    0    -1
+$EndComp
+Wire Wire Line
+	5650 1300 5700 1300
+Wire Wire Line
+	5700 1300 5700 1500
+Wire Wire Line
+	5650 1500 5700 1500
+Connection ~ 5700 1500
+Wire Wire Line
+	5700 1500 5700 1650
+Wire Wire Line
+	5000 900  5000 800
+Wire Wire Line
+	5000 800  5700 800
+Wire Wire Line
+	5700 800  5700 1050
+Connection ~ 5700 1300
+Wire Wire Line
+	5650 1050 5700 1050
+Connection ~ 5700 1050
+Wire Wire Line
+	5700 1050 5700 1300
+Text GLabel 5250 750  1    50   Input ~ 0
+SDA
+Text GLabel 4850 750  1    50   Input ~ 0
+SCL
+Wire Wire Line
+	4850 900  4850 750
+Wire Wire Line
+	5250 900  5250 750
+$Comp
+L power:+3.3V #PWR0112
+U 1 1 5DE486D2
+P 5400 700
+F 0 "#PWR0112" H 5400 550 50  0001 C CNN
+F 1 "+3.3V" H 5415 873 50  0000 C CNN
+F 2 "" H 5400 700 50  0001 C CNN
+F 3 "" H 5400 700 50  0001 C CNN
+	1    5400 700
+	-1   0    0    -1
+$EndComp
+$Comp
+L Device:C C10
+U 1 1 5DE4E3B5
+P 5600 700
+F 0 "C10" V 5450 900 50  0000 C CNN
+F 1 "100nF" V 5439 700 50  0000 C CNN
+F 2 "Capacitor_SMD:C_0603_1608Metric_Pad1.05x0.95mm_HandSolder" H 5638 550 50  0001 C CNN
+F 3 "~" H 5600 700 50  0001 C CNN
+	1    5600 700
+	0    1    1    0
+$EndComp
+Wire Wire Line
+	5150 900  5250 900
+Wire Wire Line
+	5400 900  5400 700
+Connection ~ 5250 900
+Wire Wire Line
+	5250 900  5400 900
+Wire Wire Line
+	5400 700  5450 700
+Connection ~ 5400 700
+$Comp
+L power:GND #PWR0113
+U 1 1 5DE58067
+P 5750 700
+F 0 "#PWR0113" H 5750 450 50  0001 C CNN
+F 1 "GND" H 5755 527 50  0000 C CNN
+F 2 "" H 5750 700 50  0001 C CNN
+F 3 "" H 5750 700 50  0001 C CNN
+	1    5750 700
+	0    -1   -1   0
+$EndComp
+NoConn ~ 4700 900
+NoConn ~ 5600 7300
+NoConn ~ 5700 7300
+NoConn ~ 5800 7300
+NoConn ~ 6000 7700
 $EndSCHEMATC
