File: Secondcansat.sch (KiCad schematic (older format))
At the start: 55 parts, among them IC1 XBP9B-XCWT-001, J1 OpenlogBreakout, J10 SDA, J11 5V, J12 Tx, J13 Rx, J14 Battery_Holder_keystone 1079, J15 USB_B_Mini, J16 coinBattery, J2 Camera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

Commit message: Did some stuff
Parts:
- added J?: RBF, symbol valkyrie_symbols:RBF
- added Q? (x2): Q_NMOS_BSS138, Package_TO_SOT_SMD:SOT-23, symbol Device:Q_NMOS_DGS
- added R? (x2): 10kohm, Resistor_SMD:R_0603_1608Metric_Pad1.05x0.95mm_HandSolder, symbol Device:R
- added Servo?: Servo_Adafruit_FS90R, Connector_PinSocket_2.54mm:PinSocket_1x03_P2.54mm_Vertical, symbol Connector_Generic:Conn_01x03
- added Servo?: Servo_Adafruit_SG92R, Connector_PinSocket_2.54mm:PinSocket_1x03_P2.54mm_Vertical, symbol Connector_Generic:Conn_01x03
- Servo1: value Servo_Adafruit_1142 -> Servo_Adafruit_FS90R
Connections:
- net labels added: Buzzer, TCD1
- wire segments 132 -> 142
Changed lines of the file:
@@
 P 4700 2750
 F 0 "Servo1" V 4850 2850 50  0000 R CNN
-F 1 "Servo_Adafruit_1142" V 4950 2850 50  0000 R CNN
+F 1 "Servo_Adafruit_FS90R" V 4950 2850 50  0000 R CNN
 F 2 "Connector_PinSocket_2.54mm:PinSocket_1x03_P2.54mm_Vertical" H 4700 2750 50  0001 C CNN
 F 3 "~" H 4700 2750 50  0001 C CNN
@@
 $EndComp
 $Sheet
-S 4300 4850 2750 1500
+S 4300 4900 2750 1500
 U 5C85E42A
 F0 "xbee" 50
@@
 Text GLabel 3350 4300 2    50   Input ~ 0
 MoterRIN2
-Text GLabel 6150 6650 0    50   Input ~ 0
+Text GLabel 6050 4750 0    50   Input ~ 0
 TC_PD0
 Text GLabel 1950 5200 0    50   Input ~ 0
@@
 Connection ~ 1300 850
 Wire Wire Line
-	900  1300 900  900
-Wire Wire Line
 	900  900  1200 900
 Wire Wire Line
@@
 NoConn ~ 5800 7300
 NoConn ~ 6000 7700
+$Comp
+L valkyrie_symbols:RBF J?
+U 1 1 5E18D93B
+P 1100 1050
+F 0 "J?" H 1180 1042 50  0000 L CNN
+F 1 "RBF" H 1180 951 50  0000 L CNN
+F 2 "" H 1100 1050 50  0001 C CNN
+F 3 "~" H 1100 1050 50  0001 C CNN
+	1    1100 1050
+	1    0    0    -1
+$EndComp
+Wire Wire Line
+	900  1050 900  900
+Wire Wire Line
+	900  1150 900  1300
+$Comp
+L Connector_Generic:Conn_01x03 Servo?
+U 1 1 5E1D8E04
+P 5400 4100
+F 0 "Servo?" V 5550 4200 50  0000 R CNN
+F 1 "Servo_Adafruit_FS90R" V 5650 4200 50  0000 R CNN
+F 2 "Connector_PinSocket_2.54mm:PinSocket_1x03_P2.54mm_Vertical" H 5400 4100 50  0001 C CNN
+F 3 "~" H 5400 4100 50  0001 C CNN
+	1    5400 4100
+	0    -1   -1   0
+$EndComp
+$Comp
+L Connector_Generic:Conn_01x03 Servo?
+U 1 1 5E1DDD15
+P 5950 4150
+F 0 "Servo?" V 6100 4250 50  0000 R CNN
+F 1 "Servo_Adafruit_SG92R" V 6050 3950 50  0000 R CNN
+F 2 "Connector_PinSocket_2.54mm:PinSocket_1x03_P2.54mm_Vertical" H 5950 4150 50  0001 C CNN
+F 3 "~" H 5950 4150 50  0001 C CNN
+	1    5950 4150
+	0    -1   -1   0
+$EndComp
+$Comp
+L power:GND #PWR?
+U 1 1 5E1E2F92
+P 5500 4300
+F 0 "#PWR?" H 5500 4050 50  0001 C CNN
+F 1 "GND" H 5350 4250 50  0000 C CNN
+F 2 "" H 5500 4300 50  0001 C CNN
+F 3 "" H 5500 4300 50  0001 C CNN
+	1    5500 4300
+	1    0    0    -1
+$EndComp
+$Comp
+L Device:Q_NMOS_DGS Q?
+U 1 1 5E1E316D
+P 5200 4500
+F 0 "Q?" H 5100 4350 50  0000 L CNN
+F 1 "Q_NMOS_BSS138" H 5050 4150 50  0000 L CNN
+F 2 "Package_TO_SOT_SMD:SOT-23" H 5400 4600 50  0001 C CNN
+F 3 "~" H 5200 4500 50  0001 C CNN
+	1    5200 4500
+	1    0    0    -1
+$EndComp
+$Comp
+L Device:R R?
+U 1 1 5E1ECE40
+P 5000 4650
+F 0 "R?" H 5070 4696 50  0000 L CNN
+F 1 "10kohm" H 5070 4605 50  0000 L CNN
+F 2 "Resistor_SMD:R_0603_1608Metric_Pad1.05x0.95mm_HandSolder" V 4930 4650 50  0001 C CNN
+F 3 "~" H 5000 4650 50  0001 C CNN
+	1    5000 4650
+	1    0    0    -1
+$EndComp
+$Comp
+L power:GND #PWR?
+U 1 1 5E1ED159
+P 5000 4800
+F 0 "#PWR?" H 5000 4550 50  0001 C CNN
+F 1 "GND" V 5005 4672 50  0000 R CNN
+F 2 "" H 5000 4800 50  0001 C CNN
+F 3 "" H 5000 4800 50  0001 C CNN
+	1    5000 4800
+	0    1    1    0
+$EndComp
+$Comp
+L power:+5V #PWR?
+U 1 1 5E1F24A0
+P 5400 4300
+F 0 "#PWR?" H 5400 4150 50  0001 C CNN
+F 1 "+5V" H 5450 4450 50  0000 C CNN
+F 2 "" H 5400 4300 50  0001 C CNN
+F 3 "" H 5400 4300 50  0001 C CNN
+	1    5400 4300
+	-1   0    0    1
+$EndComp
+$Comp
+L power:GND #PWR?
+U 1 1 5E1F2695
+P 5300 4700
+F 0 "#PWR?" H 5300 4450 50  0001 C CNN
+F 1 "GND" V 5400 4700 50  0000 R CNN
+F 2 "" H 5300 4700 50  0001 C CNN
+F 3 "" H 5300 4700 50  0001 C CNN
+	1    5300 4700
+	1    0    0    -1
+$EndComp
+$Comp
+L power:GND #PWR?
+U 1 1 5E1FC399
+P 6050 4350
+F 0 "#PWR?" H 6050 4100 50  0001 C CNN
+F 1 "GND" H 5900 4300 50  0000 C CNN
+F 2 "" H 6050 4350 50  0001 C CNN
+F 3 "" H 6050 4350 50  0001 C CNN
+	1    6050 4350
+	1    0    0    -1
+$EndComp
+$Comp
+L power:+5V #PWR?
+U 1 1 5E1FC41C
+P 5950 4350
+F 0 "#PWR?" H 5950 4200 50  0001 C CNN
+F 1 "+5V" H 6000 4500 50  0000 C CNN
+F 2 "" H 5950 4350 50  0001 C CNN
+F 3 "" H 5950 4350 50  0001 C CNN
+	1    5950 4350
+	-1   0    0    1
+$EndComp
+$Comp
+L Device:Q_NMOS_DGS Q?
+U 1 1 5E1FC5EE
+P 6400 4550
+F 0 "Q?" H 6300 4400 50  0000 L CNN
+F 1 "Q_NMOS_BSS138" H 6600 4350 50  0000 L CNN
+F 2 "Package_TO_SOT_SMD:SOT-23" H 6600 4650 50  0001 C CNN
+F 3 "~" H 6400 4550 50  0001 C CNN
+	1    6400 4550
+	1    0    0    -1
+$EndComp
+$Comp
+L Device:R R?
+U 1 1 5E201A5C
+P 6200 4700
+F 0 "R?" H 6270 4746 50  0000 L CNN
+F 1 "10kohm" H 6270 4655 50  0000 L CNN
+F 2 "Resistor_SMD:R_0603_1608Metric_Pad1.05x0.95mm_HandSolder" V 6130 4700 50  0001 C CNN
+F 3 "~" H 6200 4700 50  0001 C CNN
+	1    6200 4700
+	1    0    0    -1
+$EndComp
+$Comp
+L power:GND #PWR?
+U 1 1 5E201BB8
+P 6200 4850
+F 0 "#PWR?" H 6200 4600 50  0001 C CNN
+F 1 "GND" V 6205 4722 50  0000 R CNN
+F 2 "" H 6200 4850 50  0001 C CNN
+F 3 "" H 6200 4850 50  0001 C CNN
+	1    6200 4850
+	0    1    1    0
+$EndComp
+Text GLabel 1950 5600 0    50   Input ~ 0
+TCD1
+Text GLabel 5000 4500 0    50   Input ~ 0
+TCD1
+Wire Wire Line
+	6050 4750 6100 4750
+Text GLabel 6150 6700 0    50   Input ~ 0
+Buzzer
+Text GLabel 1950 5300 0    50   Input ~ 0
+Buzzer
+Wire Wire Line
+	6100 4550 6200 4550
+Wire Wire Line
+	6100 4550 6100 4750
+Connection ~ 6200 4550
+Wire Wire Line
+	6100 4550 5850 4550
+Wire Wire Line
+	5850 4550 5850 4350
+Connection ~ 6100 4550
+$Comp
+L power:GND #PWR?
+U 1 1 5E2279EF
+P 9700 4000
+F 0 "#PWR?" H 9700 3750 50  0001 C CNN
+F 1 "GND" V 9705 3872 50  0000 R CNN
+F 2 "" H 9700 4000 50  0001 C CNN
+F 3 "" H 9700 4000 50  0001 C CNN
+	1    9700 4000
+	0    1    1    0
+$EndComp
+Wire Wire Line
+	9700 4000 9750 4000
+Wire Wire Line
+	9750 4000 9750 3900
+Wire Wire Line
+	9750 3900 9800 3900
+Connection ~ 9750 4000
+Wire Wire Line
+	9750 4000 9800 4000
+Text GLabel 9800 3700 0    50   Input ~ 0
+SDA
+Text GLabel 9800 3800 0    50   Input ~ 0
+SCL
+$Comp
+L power:+5V #PWR?
+U 1 1 5E232E27
+P 9800 3600
+F 0 "#PWR?" H 9800 3450 50  0001 C CNN
+F 1 "+5V" H 9850 3750 50  0000 C CNN
+F 2 "" H 9800 3600 50  0001 C CNN
+F 3 "" H 9800 3600 50  0001 C CNN
+	1    9800 3600
+	0    -1   -1   0
+$EndComp
 $EndSCHEMATC
