File: Secondcansat.sch (KiCad schematic (older format))
At the start: 62 parts, among them IC1 XBP9B-XCWT-001, J1 OpenlogBreakout, J10 SDA, J11 5V, J12 Tx, J13 Rx, J14 Battery_Holder_keystone 1079, J15 USB_B_Mini, J16 coinBattery, J2 Camera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

Commit message: Did pcb
Parts:
- removed R17: 10kohm, Resistor_SMD:R_0603_1608Metric_Pad1.05x0.95mm_HandSolder, symbol Device:R
- C1, C5: footprint Capacitor_SMD:C_1206_3216Metric_Pad1.42x1.75mm_HandSolder -> Capacitor_Tantalum_SMD:CP_EIA-6032-15_Kemet-U
- C10, C14, C2, C3, C4, C7, C8: footprint Capacitor_SMD:C_0603_1608Metric_Pad1.05x0.95mm_HandSolder -> Capacitor_SMD:C_0603_1608Metric
- C6: footprint Capacitor_SMD:C_0805_2012Metric_Pad1.15x1.40mm_HandSolder -> Capacitor_SMD:C_0603_1608Metric
- C9: footprint Capacitor_SMD:C_1206_3216Metric_Pad1.42x1.75mm_HandSolder -> Capacitor_SMD:C_0603_1608Metric
- IC1: footprint CanSAT2ndtry:XBP9BXCWT001_2 -> valkyrie_footprints:XBP9BXCWT001
- IMU1: footprint CanSAT2ndtry:BNO055breakout -> valkyrie_footprints:BNO055breakout
- J1: footprint Connector_PinSocket_2.54mm:PinSocket_1x06_P2.54mm_Vertical -> valkyrie_footprints:PinHeader_1x06_P2.54mm_Vertical
- J14: footprint CanSAT2ndtry:BatteryHolder -> valkyrie_footprints:BatteryHolder
- J16: footprint CanSAT2ndtry:coin_Battery_120591-1 -> valkyrie_footprints:coin_Battery_120591-1
- J2: footprint Connector_PinSocket_2.54mm:PinSocket_1x03_P2.54mm_Vertical -> valkyrie_footprints:PinHeader_1x03_P2.54mm_Vertical
- J3: footprint CanSAT2ndtry:MS5607 -> valkyrie_footprints:pressure_MS5607
- J4: footprint Connector_PinSocket_1.27mm:PinSocket_2x03_P1.27mm_Vertical -> valkyrie_footprints:PDI connector
- J5: renamed from J?; footprint (none) -> valkyrie_footprints:RBF_SS0750301F020P1A
- J6: footprint CanSAT2ndtry:CAM-M8Q -> valkyrie_footprints:CAM-M8Q
- MCU1: footprint CanSAT2ndtry:ATXMEGA128A4U-AU -> valkyrie_footprints:ATXMEGA128A4U-AU
- Q1, Q2, Q3, Q4: footprint Package_TO_SOT_SMD:SOT-23 -> valkyrie_footprints:SOT-23_PMOS
- Q5, Q6: renamed from Q?; footprint Package_TO_SOT_SMD:SOT-23 -> valkyrie_footprints:SOT-23_PMOS
- R1: footprint Resistor_SMD:R_1206_3216Metric -> Resistor_SMD:R_0603_1608Metric_Pad1.05x0.95mm_HandSolder
- R10, R8, R9: footprint Capacitor_SMD:C_0805_2012Metric -> Resistor_SMD:R_0603_1608Metric_Pad1.05x0.95mm_HandSolder
- R2: footprint Resistor_SMD:R_0805_2012Metric_Pad1.15x1.40mm_HandSolder -> Resistor_SMD:R_0603_1608Metric_Pad1.05x0.95mm_HandSolder
- U1: footprint CanSAT2ndtry:VR_TPS7A7001DDAR -> valkyrie_footprints:VR_TPS7A7001DDAR
- U2: footprint (none) -> valkyrie_footprints:Diff_Press
- U3: footprint (none) -> Connector_PinSocket_2.54mm:PinSocket_1x05_P2.54mm_Vertical
- VR1: footprint CanSAT2ndtry:VR_296-50411-1-ND -> valkyrie_footprints:Vreg3.3
- buzzer1: footprint Connector_PinSocket_2.54mm:PinSocket_1x02_P2.54mm_Vertical -> valkyrie_footprints:Buzzer
- gave numbers to parts that had none: 4
Connections:
- wire segments 146 -> 147

Commit message: reversed source and drain in the Pchannel mosfet
Connections:
- wire segments 147 -> 149
Changed lines of the file:
@@
 L power:+6V #PWR01
 U 1 1 5C8F95C8
-P 900 1700
-F 0 "#PWR01" H 900 1550 50  0001 C CNN
-F 1 "+6V" H 915 1873 50  0000 C CNN
-F 2 "" H 900 1700 50  0001 C CNN
-F 3 "" H 900 1700 50  0001 C CNN
-	1    900  1700
-	-1   0    0    1
+P 900 1300
+F 0 "#PWR01" H 900 1150 50  0001 C CNN
+F 1 "+6V" H 915 1473 50  0000 C CNN
+F 2 "" H 900 1300 50  0001 C CNN
+F 3 "" H 900 1300 50  0001 C CNN
+	1    900  1300
+	0    1    1    0
 $EndComp
 $Comp
@@
 Wire Wire Line
 	900  1050 900  900
-Wire Wire Line
-	900  1150 900  1300
 $Comp
 L Connector_Generic:Conn_01x03 Servo2
@@
 	5400 850  5400 700
 Connection ~ 5400 700
+Wire Wire Line
+	900  1150 800  1150
+Wire Wire Line
+	800  1150 800  1700
+Wire Wire Line
+	800  1700 900  1700
 $EndSCHEMATC
